File: eagle1/eagle1.kicad_pcb (KiCad board)
At the start: 2 copper layers, 2 parts, among them J1 USB-C Plug, J2 USB-C Plug

Commit message: layout wip
Connections:
- net Net-(J1-CC1) renamed /CC1
- net Net-(J1-GND-PadA1) renamed /GND
- net Net-(J1-SBU1) renamed /SBU1
- J1 pad A11: unconnected-(J1-RX2+-PadA11) -> /CC2
- J1 pad A3: unconnected-(J1-TX1--PadA3) -> /SBU2
- J1 pad A4: Net-(J1-VBUS-PadA4) -> /VBUS
- J1 pad A9: Net-(J1-VBUS-PadA4) -> /VBUS
- J1 pad B10: unconnected-(J1-RX1--PadB10) -> /SBU2
- J1 pad B11: unconnected-(J1-RX1+-PadB11) -> /VBUS
- J1 pad B2: unconnected-(J1-TX2+-PadB2) -> /CC2
- J1 pad B3: unconnected-(J1-TX2--PadB3) -> /CC2
- J1 pad B4: Net-(J1-VBUS-PadA4) -> /VBUS
- J1 pad B5: Net-(J1-CC2) -> /CC2
- J1 pad B6: /D+ -> unconnected-(J1-D+-PadB6)
- J1 pad B7: /D- -> unconnected-(J1-D--PadB7)
- J1 pad B8: Net-(J1-SBU2) -> /SBU2
- J1 pad B9: Net-(J1-VBUS-PadA4) -> /VBUS
- J2 pad A4: Net-(J1-VBUS-PadA4) -> /VBUS
- J2 pad A9: Net-(J1-VBUS-PadA4) -> /VBUS
- J2 pad B10: unconnected-(J2-RX1--PadB10) -> /SBU2
- J2 pad B11: unconnected-(J2-RX1+-PadB11) -> /VBUS
- J2 pad B2: unconnected-(J2-TX2+-PadB2) -> /CC2
- J2 pad B3: unconnected-(J2-TX2--PadB3) -> /CC2
- J2 pad B4: Net-(J1-VBUS-PadA4) -> /VBUS
- J2 pad B5: Net-(J1-CC2) -> /CC2
- J2 pad B6: /D+ -> unconnected-(J2-D+-PadB6)
- J2 pad B7: /D- -> unconnected-(J2-D--PadB7)
- J2 pad B8: Net-(J1-SBU2) -> /SBU2
- J2 pad B9: Net-(J1-VBUS-PadA4) -> /VBUS
Routing:
- net /VBUS: track 0.00 -> 2382.7 mm, vias 0 -> 7
- net /GND: track 1209.3 -> 14.8 mm, vias 0 -> 4
- net Net-(J1-VBUS-PadA4): track 1193.2 -> 0.00 mm, vias 1 -> 0
- net /CC2: track 0.00 -> 601.4 mm
- net /SBU2: track 0.00 -> 599.6 mm
- net /CC1: track 0.00 -> 595.8 mm, vias 0 -> 1
- net /SBU1: track 0.00 -> 595.8 mm, vias 0 -> 1
- added copper zone on B.Cu, net /GND
- added copper zone on F.Cu, net /GND
- added copper zone on B.Cu, net /VBUS
- added copper zone on F.Cu, net /VBUS
Other:
- board outline added: 600 x 11.4 mm

Commit message: Add info for FR4 stiffener
Other:
- board text added: "FR4 stiffener to be used PCB ends."
Changed lines of the file:
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@@
       (net 11 "/GND") (thermal_bridge_angle 45))
   )
+  (gr_line (start 45 44.345) (end 45 55.7)
+    (stroke (width 0.15) (type default)) (layer "Dwgs.User"))
+  (gr_line (start 25 44.345) (end 45 44.345)
+    (stroke (width 0.15) (type default)) (layer "Dwgs.User"))
+  (gr_line (start 625 44.345) (end 605 44.345)
+    (stroke (width 0.15) (type default)) (layer "Dwgs.User"))
+  (gr_line (start 625 55.7) (end 625 44.345)
+    (stroke (width 0.15) (type default)) (layer "Dwgs.User"))
+  (gr_line (start 45 55.7) (end 25 55.7)
+    (stroke (width 0.15) (type default)) (layer "Dwgs.User"))
+  (gr_line (start 25 55.7) (end 25 44.345)
+    (stroke (width 0.15) (type default)) (layer "Dwgs.User"))
+  (gr_line (start 605 44.345) (end 605 55.7)
+    (stroke (width 0.15) (type default)) (layer "Dwgs.User"))
+  (gr_line (start 605 55.7) (end 625 55.7)
+    (stroke (width 0.15) (type default)) (layer "Dwgs.User"))
   (gr_line (start 625 55.7) (end 615 55.7)
     (stroke (width 0.1) (type default)) (layer "Edge.Cuts"))
@@
   (gr_line (start 45.95 55.7) (end 25 55.7)
     (stroke (width 0.1) (type default)) (layer "Edge.Cuts"))
+  (gr_text "FR4 stiffener to be used\nPCB ends." (at 25.1 35.45) (layer "Dwgs.User")
+    (effects (font (size 1 1) (thickness 0.15)) (justify left bottom))
+  )
+  (gr_text "FR4 stiffener to be used\nPCB ends." (at 605.55 36.95) (layer "Dwgs.User")
+    (effects (font (size 1 1) (thickness 0.15)) (justify left bottom))
+  )
+  (dimension (type aligned) (layer "Dwgs.User")
+    (pts (xy 25 44.35) (xy 45 44.35))
+    (height -3.15)
+    (gr_text "20.0000 mm" (at 35 40.05) (layer "Dwgs.User")
+      (effects (font (size 1 1) (thickness 0.15)))
+    )
+    (format (prefix "") (suffix "") (units 3) (units_format 1) (precision 4))
+    (style (thickness 0.15) (arrow_length 1.27) (text_position_mode 0) (extension_height 0.58642) (extension_offset 0.5) keep_text_aligned)
+  )
+  (dimension (type aligned) (layer "Dwgs.User")
+    (pts (xy 45 44.345) (xy 45 55.7))
+    (height -2.7)
+    (gr_text "11.3550 mm" (at 46.55 50.0225 90) (layer "Dwgs.User")
+      (effects (font (size 1 1) (thickness 0.15)))
+    )
+    (format (prefix "") (suffix "") (units 3) (units_format 1) (precision 4))
+    (style (thickness 0.15) (arrow_length 1.27) (text_position_mode 0) (extension_height 0.58642) (extension_offset 0.5) keep_text_aligned)
+  )
+  (dimension (type aligned) (layer "Dwgs.User")
+    (pts (xy 605 44.345) (xy 605 55.7))
+    (height 2.8)
+    (gr_text "11.3550 mm" (at 601.05 50.0225 90) (layer "Dwgs.User")
+      (effects (font (size 1 1) (thickness 0.15)))
+    )
+    (format (prefix "") (suffix "") (units 3) (units_format 1) (precision 4))
+    (style (thickness 0.15) (arrow_length 1.27) (text_position_mode 0) (extension_height 0.58642) (extension_offset 0.5) keep_text_aligned)
+  )
+  (dimension (type aligned) (layer "Dwgs.User")
+    (pts (xy 605 44.345) (xy 625 44.345))
+    (height -2.495)
+    (gr_text "20.0000 mm" (at 615 40.7) (layer "Dwgs.User")
+      (effects (font (size 1 1) (thickness 0.15)))
+    )
+    (format (prefix "") (suffix "") (units 3) (units_format 1) (precision 4))
+    (style (thickness 0.15) (arrow_length 1.27) (text_position_mode 0) (extension_height 0.58642) (extension_offset 0.5) keep_text_aligned)
+  )
   (segment (start 26.4 54.275) (end 25.7 53.575) (width 0.3) (layer "F.Cu") (net 11))
   (segment (start 25.7 53.575) (end 25.7 53.28) (width 0.3) (layer "F.Cu") (net 11))

Commit message: Suggested layout adjustments.
Routing:
- net /VBUS: track 2382.7 -> 1198.4 mm, vias 7 -> 11
- net /GND: track 14.8 -> 3.35 mm

Commit message: Beef up VBUS cross-connections a bit more.
Routing:
- net /GND: track 3.35 -> 0.00 mm
- net /VBUS: track 1198.4 -> 1199.1 mm, vias 11 -> 16
Changed lines of the file:
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@@
     (style (thickness 0.15) (arrow_length 1.27) (text_position_mode 0) (extension_height 0.58642) (extension_offset 0.5) keep_text_aligned)
   )
-  (segment (start 26.4 54.275) (end 25.7 53.575) (width 0.3) (layer "F.Cu") (net 11))
-  (segment (start 25.7 53.575) (end 25.7 53.28) (width 0.3) (layer "F.Cu") (net 11))
-  (segment (start 26.23 52.75) (end 27.15 52.75) (width 0.3) (layer "F.Cu") (net 11))
-  (segment (start 25.7 53.28) (end 26.23 52.75) (width 0.3) (layer "F.Cu") (net 11))
-  (segment (start 26.8 54.275) (end 26.4 54.275) (width 0.3) (layer "F.Cu") (net 11))
   (via (at 31.15 54.3) (size 0.8) (drill 0.4) (layers "F.Cu" "B.Cu") (free) (net 11))
   (via (at 29.95 54.3) (size 0.8) (drill 0.4) (layers "F.Cu" "B.Cu") (free) (net 11))
   (via (at 29.95 55.15) (size 0.8) (drill 0.4) (layers "F.Cu" "B.Cu") (free) (net 11))
   (via (at 31.15 55.15) (size 0.8) (drill 0.4) (layers "F.Cu" "B.Cu") (free) (net 11))
-  (segment (start 28.6 48.5) (end 28.75 48.65) (width 0.5) (layer "F.Cu") (net 12))
-  (segment (start 621.75 51.25) (end 28.85 51.25) (width 0.3) (layer "F.Cu") (net 12))
+  (segment (start 27.9 48.75) (end 27.15 48.75) (width 0.3) (layer "F.Cu") (net 12))
   (segment (start 623.67 48.65) (end 623.77 48.75) (width 0.5) (layer "F.Cu") (net 12))
   (segment (start 28.85 51.25) (end 28.4 51.25) (width 0.3) (layer "F.Cu") (net 12))
-  (segment (start 28.35 48.75) (end 28.6 48.5) (width 0.3) (layer "F.Cu") (net 12))
   (segment (start 26.23 48.75) (end 27.15 48.75) (width 0.3) (layer "F.Cu") (net 12))
+  (segment (start 28.85 51.25) (end 622 51.25) (width 0.3) (layer "F.Cu") (net 12))
   (segment (start 28.4 51.25) (end 27.95 51.25) (width 0.3) (layer "F.Cu") (net 12))
-  (segment (start 27.15 48.75) (end 28.35 48.75) (width 0.3) (layer "F.Cu") (net 12))
-  (segment (start 621.75 51.25) (end 622.2 51.25) (width 0.3) (layer "F.Cu") (net 12))
-  (segment (start 28.75 48.65) (end 623.67 48.65) (width 0.5) (layer "F.Cu") (net 12))
+  (segment (start 28.1 48.55) (end 28.2 48.65) (width 0.5) (layer "F.Cu") (net 12))
+  (segment (start 28.1 48.55) (end 27.9 48.75) (width 0.3) (layer "F.Cu") (net 12))
+  (segment (start 28.2 48.65) (end 623.67 48.65) (width 0.5) (layer "F.Cu") (net 12))
   (segment (start 27.15 51.25) (end 27.95 51.25) (width 0.3) (layer "F.Cu") (net 12))
   (via (at 622 51.25) (size 0.3) (drill 0.125) (layers "F.Cu" "B.Cu") (net 12))
   (via (at 621.6 51.25) (size 0.3) (drill 0.125) (layers "F.Cu" "B.Cu") (net 12))
+  (via (at 28.8 53.3) (size 0.7) (drill 0.3) (layers "F.Cu" "B.Cu") (free) (net 12))
   (via (at 621.2 51.25) (size 0.3) (drill 0.125) (layers "F.Cu" "B.Cu") (net 12))
+  (via (at 621.9 52.45) (size 0.7) (drill 0.3) (layers "F.Cu" "B.Cu") (free) (net 12))
   (via (at 28.85 51.25) (size 0.3) (drill 0.125) (layers "F.Cu" "B.Cu") (net 12))
   (via (at 27.95 51.25) (size 0.3) (drill 0.125) (layers "F.Cu" "B.Cu") (net 12))
-  (via (at 28.5 52.45) (size 0.7) (drill 0.3) (layers "F.Cu" "B.Cu") (free) (net 12))
-  (via (at 28.5 53.2) (size 0.7) (drill 0.3) (layers "F.Cu" "B.Cu") (free) (net 12))
+  (via (at 28.1 53.3) (size 0.7) (drill 0.3) (layers "F.Cu" "B.Cu") (free) (net 12))
+  (via (at 28.1 52.45) (size 0.7) (drill 0.3) (layers "F.Cu" "B.Cu") (free) (net 12))
+  (via (at 28.8 52.45) (size 0.7) (drill 0.3) (layers "F.Cu" "B.Cu") (free) (net 12))
   (via (at 28.4 51.25) (size 0.3) (drill 0.125) (layers "F.Cu" "B.Cu") (net 12))
   (via (at 621.2 48.55) (size 0.7) (drill 0.3) (layers "F.Cu" "B.Cu") (free) (net 12))
   (via (at 621.2 52.45) (size 0.7) (drill 0.3) (layers "F.Cu" "B.Cu") (free) (net 12))
-  (via (at 28.6 48.5) (size 0.7) (drill 0.3) (layers "F.Cu" "B.Cu") (net 12))
+  (via (at 28.1 48.55) (size 0.7) (drill 0.3) (layers "F.Cu" "B.Cu") (net 12))
+  (via (at 28.8 48.55) (size 0.7) (drill 0.3) (layers "F.Cu" "B.Cu") (net 12))
+  (via (at 621.9 48.55) (size 0.7) (drill 0.3) (layers "F.Cu" "B.Cu") (free) (net 12))
   (segment (start 621.2 48.55) (end 621.2 52.45) (width 0.5) (layer "B.Cu") (net 12))
   (segment (start 25.5 51.25) (end 25.598629 51.25) (width 0.5) (layer "B.Cu") (net 12))
-  (segment (start 622.2 51.25) (end 622.85 51.25) (width 0.3) (layer "B.Cu") (net 12))
+  (segment (start 621.2 51.25) (end 622.85 51.25) (width 0.3) (layer "B.Cu") (net 12))
   (segment (start 623.77 48.75) (end 622.85 48.75) (width 0.3) (layer "B.Cu") (net 12))
   (segment (start 622.050001 50.225001) (end 622.1 50.275) (width 0.2) (layer "F.Cu") (net 13))
@@
         (xy 31.95 52.1)
         (xy 31.95 53.65)
-        (xy 27.8 53.65)
-        (xy 27.8 52.1)
+        (xy 27.75 53.65)
+        (xy 27.75 52.1)
       )
     )
@@
         (xy 25 55.75)
         (xy 28.9 55.75)
-        (xy 29 55.65)
-        (xy 29 48.15)
+        (xy 29.15 55.65)
+        (xy 29.15 48.15)
       )
     )
+  )
+  (zone (net 12) (net_name "/VBUS") (layer "B.Cu") (hatch edge 0.5)
+    (priority 6)
+    (connect_pads yes (clearance 0.2))
+    (min_thickness 0.25) (filled_areas_thickness no)
+    (fill yes (thermal_gap 0.5) (thermal_bridge_width 0.5))
+    (polygon
+      (pts
+        (xy 620.85 48.2)
+        (xy 620.85 52.8)
+        (xy 622.25 52.8)
+        (xy 622.25 51.4)
+        (xy 623.25 51.4)
+        (xy 623.25 48.2)
+      )
+    )

Commit message: Add more VBUS; update git ignore
Routing:
- net /CC2: track 601.4 -> 604.4 mm
Changed lines of the file:
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@@
   (segment (start 622.85 49.25) (end 621.846128 49.25) (width 0.25) (layer "B.Cu") (net 16))
   (segment (start 26.23 47.75) (end 27.15 47.75) (width 0.3) (layer "F.Cu") (net 17))
-  (segment (start 27.15 47.75) (end 623.77 47.75) (width 0.3) (layer "F.Cu") (net 17))
   (segment (start 624 47.75) (end 624.5 48.25) (width 0.3) (layer "F.Cu") (net 17))
+  (segment (start 27.9 47.537942) (end 27.9 46.65) (width 0.3) (layer "F.Cu") (net 17))
+  (segment (start 27.15 47.75) (end 27.687942 47.75) (width 0.3) (layer "F.Cu") (net 17))
+  (segment (start 620.272918 44.75) (end 623.272918 47.75) (width 0.3) (layer "F.Cu") (net 17))
+  (segment (start 27.687942 47.75) (end 27.9 47.537942) (width 0.3) (layer "F.Cu") (net 17))
+  (segment (start 623.272918 47.75) (end 623.77 47.75) (width 0.3) (layer "F.Cu") (net 17))
+  (segment (start 27.9 46.65) (end 29.8 44.75) (width 0.3) (layer "F.Cu") (net 17))
   (segment (start 25.73 48.25) (end 26.23 47.75) (width 0.3) (layer "F.Cu") (net 17))
+  (segment (start 29.8 44.75) (end 620.272918 44.75) (width 0.3) (layer "F.Cu") (net 17))
   (segment (start 623.77 47.75) (end 624 47.75) (width 0.3) (layer "F.Cu") (net 17))
   (segment (start 624.5 48.25) (end 624.5 49.25) (width 0.3) (layer "F.Cu") (net 17))
@@
       )
     )
+  )
+  (zone (net 12) (net_name "/VBUS") (layer "F.Cu") (hatch edge 0.5)
+    (priority 7)
+    (connect_pads (clearance 0.2))
+    (min_thickness 0.25) (filled_areas_thickness no)
+    (fill yes (mode hatch) (thermal_gap 0.5) (thermal_bridge_width 0.5) (island_removal_mode 1) (island_area_min 10)
+      (hatch_thickness 0.3) (hatch_gap 0.5) (hatch_orientation 45)
+      (hatch_border_algorithm hatch_thickness) (hatch_min_hole_area 0.3))
+    (polygon
+      (pts
+        (xy 27.85 49)
+        (xy 27.85 47.95)
+        (xy 27.95 47.85)
+        (xy 28.55 47.85)
+        (xy 28.7 47.7)
+        (xy 28.7 46.35)
+        (xy 29.95 45.1)
+        (xy 620.2 45.1)
+        (xy 622.1 47)
+        (xy 622.1 49)
+      )
+    )

Commit message: Adjust VBUS zones; Add silkscreen
Routing:
- net /VBUS: track 1199.1 -> 606.2 mm
Other:
- board text added: "FOR USE IN TESTING ONLY - DO NOT CONNECT TO HOST - DO NOT CONNECT TO ANYTHING BUT INTENDED PORTS ON TESTER/EQUIPMENT UNDER TEST"
- board text added: "TO SASSERIDES"
- board text added: "TO TYCHO"
- board text added: "仅供测试使用 - 请勿连接主机 - 请勿连接测试仪/被测设备上的指定端口以外的任何其他端口"
- board text added: "前往萨塞里德"
- board text added: "致第谷"
Changed lines of the file:
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@@
   (gr_line (start 45.95 55.7) (end 25 55.7)
     (stroke (width 0.1) (type default)) (layer "Edge.Cuts"))
+  (gr_text "仅供测试使用 - 请勿连接主机 - 请勿连接测试仪/被测设备上的指定端口以外的任何其他端口" (at 469.466664 55.1) (layer "B.SilkS")
+    (effects (font (size 2 2) (thickness 0.3)) (justify right bottom mirror))
+  )
+  (gr_text "仅供测试使用 - 请勿连接主机 - 请勿连接测试仪/被测设备上的指定端口以外的任何其他端口" (at 469.466664 48.3) (layer "B.SilkS")
+    (effects (font (size 2 2) (thickness 0.3)) (justify right bottom mirror))
+  )
+  (gr_text "仅供测试使用 - 请勿连接主机 - 请勿连接测试仪/被测设备上的指定端口以外的任何其他端口" (at 55.016664 55.1) (layer "B.SilkS")
+    (effects (font (size 2 2) (thickness 0.3)) (justify right bottom mirror))
+  )
+  (gr_text "TO TYCHO" (at 621.1 48) (layer "B.SilkS")
+    (effects (font (size 2 2) (thickness 0.3)) (justify left bottom mirror))
+  )
+  (gr_text "FOR USE IN TESTING ONLY - DO NOT CONNECT TO HOST - DO NOT CONNECT TO ANYTHING BUT INTENDED PORTS ON TESTER/EQUIPMENT UNDER TEST" (at 210.366664 48.3) (layer "B.SilkS")
+    (effects (font (size 2 2) (thickness 0.3)) (justify right bottom mirror))
+  )
+  (gr_text "仅供测试使用 - 请勿连接主机 - 请勿连接测试仪/被测设备上的指定端口以外的任何其他端口" (at 55.016664 48.3) (layer "B.SilkS")
+    (effects (font (size 2 2) (thickness 0.3)) (justify right bottom mirror))
+  )
+  (gr_text "FOR USE IN TESTING ONLY - DO NOT CONNECT TO HOST - DO NOT CONNECT TO ANYTHING BUT INTENDED PORTS ON TESTER/EQUIPMENT UNDER TEST" (at 210.366664 55.1) (layer "B.SilkS")
+    (effects (font (size 2 2) (thickness 0.3)) (justify right bottom mirror))
+  )
+  (gr_text "致第谷" (at 618.25 55) (layer "B.SilkS")
+    (effects (font (size 2 2) (thickness 0.3)) (justify left bottom mirror))
+  )
+  (gr_text "TO SASSERIDES" (at 29.3 47.25) (layer "F.SilkS")
+    (effects (font (size 1.25 1.25) (thickness 0.2)) (justify left bottom))
+  )
+  (gr_text "仅供测试使用 - 请勿连接主机 - 请勿连接测试仪/被测设备上的指定端口以外的任何其他端口" (at 469.45 55.1) (layer "F.SilkS")
+    (effects (font (size 2 2) (thickness 0.3)) (justify left bottom))
+  )
+  (gr_text "仅供测试使用 - 请勿连接主机 - 请勿连接测试仪/被测设备上的指定端口以外的任何其他端口" (at 55 48.3) (layer "F.SilkS")
+    (effects (font (size 2 2) (thickness 0.3)) (justify left bottom))
+  )
+  (gr_text "FOR USE IN TESTING ONLY - DO NOT CONNECT TO HOST - DO NOT CONNECT TO ANYTHING BUT INTENDED PORTS ON TESTER/EQUIPMENT UNDER TEST" (at 210.35 55.1) (layer "F.SilkS")
+    (effects (font (size 2 2) (thickness 0.3)) (justify left bottom))
+  )
+  (gr_text "前往萨塞里德" (at 29.1 53.6) (layer "F.SilkS")
+    (effects (font (size 1.75 1.75) (thickness 0.25)) (justify left bottom))
+  )
+  (gr_text "仅供测试使用 - 请勿连接主机 - 请勿连接测试仪/被测设备上的指定端口以外的任何其他端口" (at 469.45 48.3) (layer "F.SilkS")
+    (effects (font (size 2 2) (thickness 0.3)) (justify left bottom))
+  )
+  (gr_text "FOR USE IN TESTING ONLY - DO NOT CONNECT TO HOST - DO NOT CONNECT TO ANYTHING BUT INTENDED PORTS ON TESTER/EQUIPMENT UNDER TEST" (at 210.35 48.3) (layer "F.SilkS")
+    (effects (font (size 2 2) (thickness 0.3)) (justify left bottom))
+  )
+  (gr_text "仅供测试使用 - 请勿连接主机 - 请勿连接测试仪/被测设备上的指定端口以外的任何其他端口" (at 55 55.1) (layer "F.SilkS")
+    (effects (font (size 2 2) (thickness 0.3)) (justify left bottom))
+  )
   (gr_text "FR4 stiffener to be used\nPCB ends." (at 25.1 35.45) (layer "Dwgs.User")
     (effects (font (size 1 1) (thickness 0.15)) (justify left bottom))
@@
     (format (prefix "") (suffix "") (units 3) (units_format 1) (precision 4))
     (style (thickness 0.15) (arrow_length 1.27) (text_position_mode 0) (extension_height 0.58642) (extension_offset 0.5) keep_text_aligned)
+  )
+  (dimension (type aligned) (layer "Dwgs.User")
+    (pts (xy 45 55.7) (xy 605 55.7))
+    (height 1.95)
+    (gr_text "560.0000 mm" (at 325 58.9) (layer "Dwgs.User")
+      (effects (font (size 1 1) (thickness 0.15)))
+    )
+    (format (prefix "") (suffix "") (units 3) (units_format 1) (precision 4))
+    (style (thickness 0.15) (arrow_length 1.27) (text_position_mode 2) (extension_height 0.58642) (extension_offset 0.5) keep_text_aligned)
   )
   (via (at 31.15 54.3) (size 0.8) (drill 0.4) (layers "F.Cu" "B.Cu") (free) (net 11))
@@
   (via (at 31.15 55.15) (size 0.8) (drill 0.4) (layers "F.Cu" "B.Cu") (free) (net 11))
   (segment (start 27.9 48.75) (end 27.15 48.75) (width 0.3) (layer "F.Cu") (net 12))
-  (segment (start 623.67 48.65) (end 623.77 48.75) (width 0.5) (layer "F.Cu") (net 12))
+  (segment (start 623.57 48.55) (end 623.77 48.75) (width 0.5) (layer "F.Cu") (net 12))
   (segment (start 28.85 51.25) (end 28.4 51.25) (width 0.3) (layer "F.Cu") (net 12))
+  (segment (start 621.2 48.55) (end 623.57 48.55) (width 0.5) (layer "F.Cu") (net 12))
   (segment (start 26.23 48.75) (end 27.15 48.75) (width 0.3) (layer "F.Cu") (net 12))
   (segment (start 28.85 51.25) (end 622 51.25) (width 0.3) (layer "F.Cu") (net 12))
@@
   (segment (start 28.1 48.55) (end 28.2 48.65) (width 0.5) (layer "F.Cu") (net 12))
   (segment (start 28.1 48.55) (end 27.9 48.75) (width 0.3) (layer "F.Cu") (net 12))
-  (segment (start 28.2 48.65) (end 623.67 48.65) (width 0.5) (layer "F.Cu") (net 12))
   (segment (start 27.15 51.25) (end 27.95 51.25) (width 0.3) (layer "F.Cu") (net 12))
   (via (at 622 51.25) (size 0.3) (drill 0.125) (layers "F.Cu" "B.Cu") (net 12))
@@
     (polygon
       (pts
-        (xy 621.5 52.1)
-        (xy 621.5 55.7)
+        (xy 618 52.1)
+        (xy 618 55.7)
         (xy 31.95 55.7)
         (xy 31.95 52.1)
@@
     (polygon
       (pts
-        (xy 27.85 49)
-        (xy 27.85 47.95)
-        (xy 27.95 47.85)
-        (xy 28.55 47.85)
-        (xy 28.7 47.7)
-        (xy 28.7 46.35)
-        (xy 29.95 45.1)
-        (xy 620.2 45.1)
-        (xy 622.1 47)
-        (xy 622.1 49)
+        (xy 32 49)
+        (xy 32 47.95)
+        (xy 32 47.85)
+        (xy 32 47.85)
+        (xy 32 47.7)
+        (xy 32 46.35)
+        (xy 32 45.1)
+        (xy 618 45.1)
+        (xy 618 45.733105)
+        (xy 618 49)
       )
     )
@@
   )
   (zone (net 12) (net_name "/VBUS") (layer "F.Cu") (hatch edge 0.5)
+    (priority 9)
+    (connect_pads (clearance 0.2))
+    (min_thickness 0.25) (filled_areas_thickness no)
+    (fill yes (thermal_gap 0.5) (thermal_bridge_width 0.5) (island_removal_mode 1) (island_area_min 10))
+    (polygon
+      (pts
+        (xy 618 49)
+        (xy 624.15 49)
+        (xy 624.15 48.65)
+        (xy 623.5 48)
+        (xy 623.1 48)
+        (xy 620.194517 45.1)
+        (xy 618 45.1)
+      )
+    )
+  )
+  (zone (net 12) (net_name "/VBUS") (layer "F.Cu") (hatch edge 0.5)
+    (priority 8)
+    (connect_pads (clearance 0.2))
+    (min_thickness 0.25) (filled_areas_thickness no)
+    (fill yes (thermal_gap 0.5) (thermal_bridge_width 0.5) (island_removal_mode 1) (island_area_min 10))
+    (polygon
+      (pts
+        (xy 32 49)
+        (xy 27.6 49)
+        (xy 27.6 47.3)
+        (xy 29.8 45.1)
+        (xy 32 45.1)
+      )
+    )
+  )
+  (zone (net 12) (net_name "/VBUS") (layer "F.Cu") (hatch edge 0.5)
     (priority 2)
     (connect_pads yes (clearance 0.2))
@@
         (xy 625.05 50.7)
         (xy 625.05 55.7)
-        (xy 620.85 55.7)
-        (xy 620.85 51.15)
+        (xy 618 55.7)
+        (xy 618 50.7)
         (xy 621.3 50.7)
       )
