File: eagle1/eagle1.kicad_pcb (KiCad board)
At the start: 2 copper layers, 600 x 11.4 mm, 2 parts, among them J1 USB-C Plug, J2 USB-C Plug

Commit message: Move stiffener specs to own layers; add Fab specs
Other:
- board text added: "FR4 stiffener to be used at PCB ends."
- board text added: "order of copper/non-copper layers: Layer 1 (non-copper): F.Stiffiner Layer 2 (copper): F.Cu Layer 3 (copper): B.Cu Layer 4 (non-copper): B.Stiffiner PCB description: 2 layer PCB 0.2224 mm Copper 1: 0.035 mm Dielectric 1: polymide 0.10160 mm Copper 2: 0.035 mm polymide substrate with Er=3.2 FR4 Stiffener required differential microstrip impedance: 7 mil trace, 7 mil space: 90 ohm (±10%) two sided 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"
- board text removed: "FR4 stiffener to be used PCB ends."

Commit message: Move traces away from D+/- traces
Routing:
- net /VBUS: track 606.2 -> 607.9 mm
- net /CC2: track 604.4 -> 603.9 mm

Commit message: Fix silkscreen
Other:
- board text added: "Eagle rev1.0.0"

Commit message: Adapt for PCBWay 0.2mm flex stackup with 400mm length.
Parts:
- moved J2 200.0 mm to (425.0, 50.0)
Routing:
- net /VBUS: track 607.9 -> 399.9 mm
- net /D-: track 595.8 -> 395.8 mm
- net /D+: track 595.8 -> 395.8 mm
- net /SBU2: track 600.0 -> 400.0 mm
- net /CC2: track 603.9 -> 403.9 mm
- net /CC1: track 596.1 -> 396.1 mm
- net /SBU1: track 595.9 -> 396.1 mm
Other:
- board size 600 x 11.4 mm -> 400 x 11.4 mm
- board text added: "2-layer flex PCB: coverlay both sides stiffeners both sides silkscreen both sides Stackup: 600um FR4 stiffener (F.Stiffener) 25um Polyimide coverlay (F.Mask) 25um Adhesive 18um Copper (24um finished) (F.Cu) 20um Adhesive 25um Polyimide core 20um Adhesive 18um Copper (24um finished) (B.Cu) 25um Adhesive 25um Polyimide coverlay (B.Mask) 600um FR4 stiffener (B.Stiffener) Impedance control: 90 ohm di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"
- board text added: "Eagle r1.0.0"
- board text added: "FR4 stiffener back side"
- board text added: "FR4 stiffener front side"
- board text removed: "COVERLAY"
- board text removed: "Eagle rev1.0.0"
- board text removed: "FR4 stiffener to be used at PCB ends."
- board text removed: "order of copper/non-copper layers: Layer 1 (non-copper): F.Stiffiner Layer 2 (copper): F.Cu Layer 3 (copper): B.Cu Layer 4 (non-copper): B.Stiffiner PCB description: 2 layer PCB 0.2224 mm Copper 1: 0.035 mm Dielectric 1: polymide 0.10160 mm Copper 2: 0.035 mm polymide substrate with Er=3.2 FR4 Stiffener required differential microstrip impedance: 7 mil trace, 7 mil space: 90 ohm (±10%) two sided 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"
